File: CAN_RPi-ZeroW.kicad_pcb (KiCad board)
At the start: 2 copper layers, 82.5 x 34 mm, 32 parts, among them J1 RJ45, J2 RJ45, J3 Raspberry_Pi_2_3, SW1 SW_SPST, U1 TJA1042T/3, U2 MCP2515-I/ST, U3 MCP16301, Y1 8MHz

Commit message: PCB errors corrected and short installation guide added to README.md
Corrected errors:
- Pin header instead of socket strip used --> wrong pin layout of Raspi connector
- STB pin of transceiver not connected --> sending of messages was not possible

Now, small 26 pin connector is used instead of full 40 pin RPi HAT connector.
Parts:
- added N1: LIBRESOLAR_LOGO, LibreSolar:LIBRESOLAR_LOGO, B.Cu at (188.8, 88.0)
- J3: value Raspberry_Pi_2_3 -> Raspberry_Pi_HAT_26p; footprint Pin_Headers:Pin_Header_Straight_2x20_Pitch2.54mm -> Socket_Strips:Socket_Strip_Straight_2x13_Pitch2.54mm
- moved N1 22.3 mm to (181.4, 94.4)
- moved LOGO1 5.97 mm to (183.6, 83.2)
- moved J3 2.50 mm to (162.0, 70.5)
Connections:
- J3 pad 18: Net-(J3-Pad18) -> /CAN_STB
- U1 pad 8: Net-(U1-Pad8) -> /CAN_STB
Routing:
- net /CAN_STB: track 0.00 -> 38.1 mm, vias 0 -> 5
- net +3V3: track 73.6 -> 68.1 mm, vias 1 -> 0
- net +5V: track 58.2 -> 61.5 mm
- net /SPI_MISO: track 28.1 -> 25.2 mm
- net /LED1: track 28.8 -> 26.3 mm, vias 2 -> 3
- net /SPI_SCLK: track 29.2 -> 26.8 mm
- net /SPI_MOSI: track 27.5 -> 25.2 mm
- net /CAN_INT: track 23.3 -> 25.4 mm, vias 2 -> 0
- net /SPI_CE0: track 30.4 -> 31.4 mm
Other:
- board size 82.5 x 34 mm -> 65 x 34 mm
- board text added: "CAN bus interface for Raspberry Pi"
- board text added: "Layout: Martin Jäger, http://libre.solar"
- board text added: "Libre Solar CAN bus interface for Raspberry Pi"
- board text removed: "Layout: Martin Jäger, http://libre.solar Made in Fabulous St. Pauli"
- board text removed: "Libre Solar CAN interface for Raspberry Pi (Zero W)"

Commit message: Pull-down resistor for transceiver STB pin added.
Parts:
- added R6: 1M, LibreSolar:R_0603_1608, B.Cu at (168.0, 74.0)
Routing:
- net /CAN_STB: track 38.1 -> 40.6 mm
- net GND: track 17.3 -> 18.3 mm, vias 12 -> 13
Changed lines of the file:
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@@
     (thickness 1.6)
     (drawings 16)
-    (tracks 290)
+    (tracks 294)
     (zones 0)
-    (modules 33)
+    (modules 34)
     (nets 45)
   )
@@
     (add_net "Net-(U2-Pad3)")
     (add_net "Net-(U2-Pad6)")
+  )
+  (module LibreSolar:R_0603_1608 (layer B.Cu)
+    (at 168 74)
+    (descr "Resistor SMD 0603, reflow soldering, Vishay (see dcrcw.pdf)")
+    (tags "resistor 0603")
+    (attr smd)
+    (fp_text reference R6 (at 0 1.4) (layer B.SilkS)
+      (effects (font (size 1 1) (thickness 0.15)) (justify mirror))
+    )
+    (fp_text value 1M (at 0 -1.5) (layer B.Fab)
+      (effects (font (size 1 1) (thickness 0.15)) (justify mirror))
+    )
+    (fp_text user %R (at 0 0) (layer B.Fab)
+      (effects (font (size 0.5 0.5) (thickness 0.075)) (justify mirror))
+    )
+    (fp_line (start -0.8 -0.4) (end -0.8 0.4) (layer B.Fab) (width 0.1))
+    (fp_line (start 0.8 -0.4) (end -0.8 -0.4) (layer B.Fab) (width 0.1))
+    (fp_line (start 0.8 0.4) (end 0.8 -0.4) (layer B.Fab) (width 0.1))
+    (fp_line (start -0.8 0.4) (end 0.8 0.4) (layer B.Fab) (width 0.1))
+    (fp_line (start 0.35 -0.55) (end -0.35 -0.55) (layer B.SilkS) (width 0.12))
+    (fp_line (start -0.35 0.55) (end 0.35 0.55) (layer B.SilkS) (width 0.12))
+    (fp_line (start -1.4 0.65) (end 1.4 0.65) (layer B.CrtYd) (width 0.05))
+    (fp_line (start -1.4 0.65) (end -1.4 -0.65) (layer B.CrtYd) (width 0.05))
+    (fp_line (start 1.4 -0.65) (end 1.4 0.65) (layer B.CrtYd) (width 0.05))
+    (fp_line (start 1.4 -0.65) (end -1.4 -0.65) (layer B.CrtYd) (width 0.05))
+    (pad 1 smd roundrect (at -0.8 0) (size 0.8 0.9) (layers B.Cu B.Paste B.Mask)(roundrect_rratio 0.2)
+      (net 44 /CAN_STB))
+    (pad 2 smd roundrect (at 0.8 0) (size 0.8 0.9) (layers B.Cu B.Paste B.Mask)(roundrect_rratio 0.2)
+      (net 18 GND))
+    (model ${KISYS3DMOD}/Resistors_SMD.3dshapes/R_0603.step
+      (at (xyz 0 0 0))
+      (scale (xyz 1 1 1))
+      (rotate (xyz 0 0 0))
+    )
   )
   (module LibreSolar:L_WE-TPC-4818 (layer B.Cu)
@@
   (segment (start 147.6 87.9) (end 147.6 89.5) (width 0.25) (layer B.Cu) (net 7))
   (segment (start 147.6 89.5) (end 146.9 90.2) (width 0.25) (layer B.Cu) (net 7))
+  (segment (start 168.8 74) (end 169.8 74) (width 0.25) (layer B.Cu) (net 18))
+  (via (at 169.8 74) (size 0.8) (drill 0.4) (layers F.Cu B.Cu) (net 18))
   (segment (start 173.2 82.8) (end 173.8 82.2) (width 0.25) (layer B.Cu) (net 18))
   (segment (start 173.2 83.4) (end 173.2 82.8) (width 0.25) (layer B.Cu) (net 18))
@@
   (segment (start 160.869999 85.530001) (end 162.675 83.725) (width 0.25) (layer B.Cu) (net 35))
   (segment (start 162.675 83.725) (end 163.65 83.725) (width 0.25) (layer B.Cu) (net 35))
+  (segment (start 167.2 74) (end 165.7 74) (width 0.25) (layer B.Cu) (net 44))
+  (segment (start 165.7 74) (end 165 73.3) (width 0.25) (layer B.Cu) (net 44))
   (segment (start 158.6 76.8) (end 158.834315 76.8) (width 0.25) (layer F.Cu) (net 44))
   (segment (start 158.834315 76.8) (end 159.4 76.8) (width 0.25) (layer F.Cu) (net 44))
